File: shema/shema.kicad_pcb (KiCad board)
At the start: 2 copper layers, 41 parts, among them J1 Power In, J2 US_01_Connector, J3 US_02_Connector, J4 US_03_Connector, J5 Valves_Connector, J6 Temp_Sensor_Connector, J7 Led_Strip_Connector, Q1 IRLML6402, Q10 IRLML6344, Q11 Q_NPN_BEC, Q12 Q_NPN_BEC, Q13 Q_NPN_BEC, Q14 Q_NPN_BEC, Q15 IRLML6344, Q16 IRLML6344, Q17 IRLML6344, Q18 IRLML6344, Q2 Q_NPN_BEC, Q3 Q_NPN_BEC, Q4 Q_NPN_BEC, Q5 Q_NPN_BEC, Q6 IRLML6344, Q7 IRLML6344, Q8 IRLML6344, Q9 IRLML6344, U1 NodeMCU1.0(ESP-12E), U2 74HC595, U3 74HC595, U4 74HC595

Commit message: first steps
Parts:
- moved Q1 309.1 mm to (-92.7, 88.9)
- moved R6 278.2 mm to (-37.3, 101.3)
- moved Q9 272.0 mm to (-51.8, 89.2)
- moved C2 260.4 mm to (-17.5, 110.0)
- moved U4 260.0 mm to (114.6, 190.8), turned to 180 degrees
- moved Q18 256.6 mm to (-79.6, 89.1)
- moved U3 255.4 mm to (114.6, 163.6), turned to 180 degrees
- moved Q10 251.5 mm to (-70.4, 88.9)
- moved Q16 250.0 mm to (-33.8, 89.7)
- moved Q3 248.4 mm to (-76.7, 78.2)
- moved Q15 247.3 mm to (-61.0, 89.2)
- moved Q7 242.1 mm to (-4.64, 90.2)
- moved Q6 239.9 mm to (-23.9, 89.7)
- moved R8 237.2 mm to (-50.3, 100.8)
- moved Q5 236.9 mm to (-66.0, 78.2)
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Connections:
- U2 pad 1: /Led_Green -> /Heater_02
- U2 pad 10: Net-(U1-Pad28) -> Net-(U1-Pad30)
- U2 pad 12: Net-(U1-Pad27) -> Net-(U1-Pad28)
- U2 pad 14: Net-(U1-Pad30) -> Net-(U1-Pad27)
- U2 pad 15: /Led_Red -> Net-(U2-Pad15)
- U2 pad 2: /Led_Blue -> /Heater_01
- U2 pad 3: /Led_White -> /Water_Pump
- U2 pad 4: /Water_Pump -> /Led_White
- U2 pad 5: /Heater_01 -> /Led_Blue
- U2 pad 6: /Heater_02 -> /Led_Green
- U2 pad 7: /Cooling -> /Led_Red
- U3 pad 1: /Valve_02 -> /Valve_04
- U3 pad 10: Net-(U1-Pad28) -> Net-(U1-Pad30)
- U3 pad 12: Net-(U1-Pad27) -> Net-(U1-Pad28)
- U3 pad 15: /Valve_01 -> /Wave_Maker
- U3 pad 3: /Valve_04 -> /Valve_02
- U3 pad 4: /Wave_Maker -> /Valve_01
- U3 pad 5: Net-(U3-Pad5) -> /Cooling
- U4 pad 10: Net-(U1-Pad28) -> Net-(U1-Pad30)
- U4 pad 12: Net-(U1-Pad27) -> Net-(U1-Pad28)
Routing:
- net Net-(U1-Pad30): track 0.00 -> 118.7 mm
- net Net-(U1-Pad29): track 0.00 -> 118.2 mm, vias 0 -> 4
- net Net-(U1-Pad28): track 0.00 -> 117.7 mm, vias 0 -> 4
- net Net-(U1-Pad27): track 0.00 -> 91.5 mm, vias 0 -> 4

Commit message: temp sensor pcb
Parts:
- Q10: value IRLML6344 -> IRLML6344TRPBFTR
- moved Q3 261.0 mm to (182.8, 106.7), turned to 270 degrees
- moved Q5 253.1 mm to (182.8, 124.5), turned to 270 degrees
- moved Q18 236.0 mm to (153.5, 125.7), turned to 180 degrees
- moved Q9 232.2 mm to (177.7, 124.5), turned to 180 degrees
- moved J5 224.0 mm to (169.9, 104.9), turned to 270 degrees
- moved Q8 222.1 mm to (177.7, 115.6), turned to 180 degrees
- moved Q14 219.5 mm to (158.6, 125.7), turned to 270 degrees
- moved J6 215.9 mm to (160.0, 155.4), turned to 270 degrees
- moved Q15 214.7 mm to (153.5, 99.1), turned to 180 degrees
- moved R3 214.7 mm to (183.0, 119.0), turned to 180 degrees
- moved Q4 211.4 mm to (182.8, 115.6), turned to 270 degrees
- moved R8 210.0 mm to (158.8, 120.3), turned to 180 degrees
- moved R2 207.8 mm to (183.0, 110.1), turned to 180 degrees
- moved Q11 205.1 mm to (158.6, 99.1), turned to 270 degrees
- moved R7 202.8 mm to (158.8, 111.4), turned to 180 degrees
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Connections:
- U2 pad 1: /Heater_02 -> /Led_Red
- U2 pad 2: /Heater_01 -> /Led_Green
- U2 pad 3: /Water_Pump -> /Led_Blue
- U2 pad 5: /Led_Blue -> /Water_Pump
- U2 pad 6: /Led_Green -> /Heater_01
- U2 pad 7: /Led_Red -> /Heater_02
- U3 pad 1: /Valve_04 -> /Valve_01
- U3 pad 15: /Wave_Maker -> Net-(U3-Pad15)
- U3 pad 2: /Valve_03 -> /Valve_02
- U3 pad 3: /Valve_02 -> /Valve_03
- U3 pad 4: /Valve_01 -> /Valve_04
- U3 pad 6: Net-(U3-Pad6) -> /Wave_Maker
Routing:
- net GND: track 0.00 -> 23.6 mm
- net Net-(J5-Pad5): track 0.00 -> 13.0 mm
- net Net-(J7-Pad5): track 0.00 -> 13.0 mm
- net Net-(J5-Pad2): track 0.00 -> 12.5 mm
- net Net-(J7-Pad2): track 0.00 -> 12.5 mm
- net /Temp_sensor: track 0.00 -> 12.0 mm
- net Net-(J5-Pad3): track 0.00 -> 8.44 mm
- net Net-(J7-Pad3): track 0.00 -> 8.44 mm
- net Net-(J5-Pad4): track 0.00 -> 8.34 mm
- net Net-(J7-Pad4): track 0.00 -> 8.34 mm
- net +3V3: track 0.00 -> 8.07 mm
- net Net-(Q14-Pad3): track 0.00 -> 6.92 mm
- net Net-(Q11-Pad3): track 0.00 -> 6.91 mm
- net Net-(Q3-Pad3): track 0.00 -> 6.87 mm
- net Net-(Q2-Pad3): track 0.00 -> 6.87 mm
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
Commit message: second version
Parts:
- removed the C1 at (-4.57, 110.0)
- removed the J7 at (145.8, 106.2)
- added C1: 100nF, Capacitor_SMD:C_0805_2012Metric, F.Cu at (178.1, 171.1)
- added C1: 100nF, Capacitor_SMD:C_0805_2012Metric, F.Cu at (106.8, 135.4)
- added C2: 100nF, Capacitor_SMD:C_0805_2012Metric, F.Cu at (195.5, 171.1)
- added C3: 100nF, Capacitor_SMD:C_0805_2012Metric, F.Cu at (212.9, 171.1)
- added J2: US_01_Connector, Connector_Molex:Molex_KK-254_AE-6410-04A_1x04_P2.54mm_Vertical, F.Cu at (236.3, 128.5)
- added J3: US_02_Connector, Connector_Molex:Molex_KK-254_AE-6410-04A_1x04_P2.54mm_Vertical, F.Cu at (224.8, 128.5)
- added J4: US_03_Connector, Connector_Molex:Molex_KK-254_AE-6410-04A_1x04_P2.54mm_Vertical, F.Cu at (213.4, 128.5)
- added J5: Valves_Connector, Connector_Molex:Molex_KK-254_AE-6410-05A_1x05_P2.54mm_Vertical, F.Cu at (190.5, 128.1)
- added J6: Temp_Sensor_Connector, Connector_Molex:Molex_KK-254_AE-6410-03A_1x03_P2.54mm_Vertical, F.Cu at (200.5, 128.5)
- added J7: Led_Strip_Connector, Connector_Molex:Molex_KK-254_AE-6410-05A_1x05_P2.54mm_Vertical, F.Cu at (176.1, 128.3)
- added J7: Led_Strip_Connector, Connector_Molex:Molex_KK-254_AE-6410-05A_1x05_P2.54mm_Vertical, F.Cu at (142.5, 148.7)
- added Q11: Q_NPN_BEC, Package_TO_SOT_SMD:SOT-23, F.Cu at (198.5, 148.2)
- added Q12: Q_NPN_BEC, Package_TO_SOT_SMD:SOT-23, F.Cu at (189.6, 148.2)
- added Q13: Q_NPN_BEC, Package_TO_SOT_SMD:SOT-23, F.Cu at (180.7, 148.2)
- added Q14: Q_NPN_BEC, Package_TO_SOT_SMD:SOT-23, F.Cu at (171.8, 148.2)
- added Q15: IRLML6344, Package_TO_SOT_SMD:SC-59, F.Cu at (198.5, 143.1)
- added Q16: IRLML6344, Package_TO_SOT_SMD:SC-59, F.Cu at (189.6, 143.1)
- added Q17: IRLML6344, Package_TO_SOT_SMD:SC-59, F.Cu at (180.7, 143.1)
- added Q18: IRLML6344, Package_TO_SOT_SMD:SC-59, F.Cu at (171.8, 143.1)
- added Q2: Q_NPN_BEC, Package_TO_SOT_SMD:SOT-23, F.Cu at (238.1, 148.1)
- added Q3: Q_NPN_BEC, Package_TO_SOT_SMD:SOT-23, F.Cu at (229.2, 148.1)
- added Q4: Q_NPN_BEC, Package_TO_SOT_SMD:SOT-23, F.Cu at (220.3, 148.1)
- added Q5: Q_NPN_BEC, Package_TO_SOT_SMD:SOT-23, F.Cu at (211.5, 148.1)
- added Q6: IRLML6344, Package_TO_SOT_SMD:SC-59, F.Cu at (238.1, 143.0)
- added Q7: IRLML6344, Package_TO_SOT_SMD:SC-59, F.Cu at (229.2, 143.0)
- added Q8: IRLML6344, Package_TO_SOT_SMD:SC-59, F.Cu at (220.3, 143.0)
- added Q9: IRLML6344, Package_TO_SOT_SMD:SC-59, F.Cu at (211.5, 143.0)
- added R1: 1K, Resistor_SMD:R_0805_2012Metric, F.Cu at (234.7, 148.3)
- added R2: 1K, Resistor_SMD:R_0805_2012Metric, F.Cu at (225.8, 148.3)
- added R3: 1K, Resistor_SMD:R_0805_2012Metric, F.Cu at (216.9, 148.3)
- added R4: 1K, Resistor_SMD:R_0805_2012Metric, F.Cu at (208.0, 148.3)
- added R5: 4.7k, Resistor_SMD:R_0805_2012Metric, F.Cu at (223.6, 171.7)
- added R6: 1K, Resistor_SMD:R_0805_2012Metric, F.Cu at (195.1, 148.4)
- added R7: 1K, Resistor_SMD:R_0805_2012Metric, F.Cu at (186.2, 148.4)
- added R8: 1K, Resistor_SMD:R_0805_2012Metric, F.Cu at (177.3, 148.4)
- added R9: 1K, Resistor_SMD:R_0805_2012Metric, F.Cu at (168.4, 148.4)
- added U1: NodeMCU1.0(ESP-12E), ESP8266:NodeMCU1.0(12-E), F.Cu at (224.0, 212.9)
- added U2: 74HC595, Package_SO:SOIC-16W_5.3x10.2mm_P1.27mm, F.Cu at (170.9, 168.5)
- added U3: 74HC595, Package_SO:SOIC-16W_5.3x10.2mm_P1.27mm, F.Cu at (188.3, 168.5)
- added U4: 74HC595, Package_SO:SOIC-16W_5.3x10.2mm_P1.27mm, F.Cu at (205.7, 168.5)
- moved Q1 401.3 mm to (308.0, 110.4)
- moved Q10 372.3 mm to (300.6, 120.4)
- moved J1 307.2 mm to (246.3, 130.0), turned to 180 degrees
- moved J2 223.0 mm to (112.8, 220.5), turned to 90 degrees
- moved J4 215.2 mm to (112.8, 197.7), turned to 90 degrees
- moved J3 205.4 mm to (112.8, 209.1), turned to 90 degrees
- moved C3 132.3 mm to (106.8, 170.2)
- moved C2 131.4 mm to (106.8, 152.8), turned to 180 degrees
- moved Q2 111.1 mm to (129.8, 195.5), turned to 90 degrees
- moved Q6 106.6 mm to (134.9, 195.5), turned to 0 degrees
- moved R1 105.3 mm to (129.6, 192.0), turned to 0 degrees
- moved Q3 95.8 mm to (129.8, 186.6), turned to 90 degrees
- moved Q7 90.6 mm to (134.9, 186.6), turned to 0 degrees
- moved R2 90.4 mm to (129.6, 183.1), turned to 0 degrees
- moved J5 85.7 mm to (142.6, 186.2), turned to 90 degrees
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Connections:
- U1 pad 20: /us_03 -> /us_01
- U1 pad 22: /us_01 -> /us_03
- U1 pad 23: /Flowmeter -> /us_trig
- U1 pad 4: /us_trig -> /Flowmeter
Routing:
- net +3V3: track 8.07 -> 129.6 mm
- net /Valve_01: track 0.00 -> 118.9 mm
- net /Valve_02: track 0.00 -> 100.9 mm
- net /Valve_04: track 0.00 -> 89.6 mm
- net /Valve_03: track 0.00 -> 87.8 mm
- net /Led_Red: track 0.00 -> 68.9 mm
- net /Led_Green: track 0.00 -> 54.8 mm
- net Net-(U1-Pad30): track 118.7 -> 165.1 mm
- net /us_trig: track 0.00 -> 45.4 mm
- net Net-(U1-Pad29): track 118.2 -> 162.3 mm, vias 4 -> 8
- net Net-(U1-Pad28): track 117.7 -> 161.6 mm, vias 4 -> 8
- net Net-(U1-Pad27): track 91.5 -> 132.0 mm, vias 4 -> 8
- net /Led_Blue: track 0.00 -> 39.0 mm
- net /Led_White: track 0.00 -> 37.4 mm
- net /Temp_sensor: track 12.0 -> 45.2 mm
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Other:
- board outline added: 190.8 x 107.7 mm

Commit message: ready
Parts:
- removed the C1 at (178.1, 171.1)
- removed the C1 at (106.8, 135.4)
- removed the C2 at (195.5, 171.1)
- removed the C2 at (106.8, 152.8)
- removed the C3 at (212.9, 171.1)
- removed the C3 at (106.8, 170.2)
- removed the J2 at (236.3, 128.5)
- removed the J2 at (112.8, 220.5)
- removed the J3 at (224.8, 128.5)
- removed the J3 at (112.8, 209.1)
- removed the J4 at (213.4, 128.5)
- removed the J4 at (112.8, 197.7)
- removed the J5 at (190.5, 128.1)
- removed the J5 at (142.6, 186.2)
- removed the J6 at (200.5, 128.5)
- removed the J6 at (112.8, 184.7)
- removed the J7 at (176.1, 128.3)
- removed the J7 at (142.5, 148.7)
- removed Q10: IRLML6344TRPBFTR, Package_TO_SOT_SMD:SC-59
- removed the Q11 at (198.5, 148.2)
- removed the Q11 at (129.7, 155.8)
- removed the Q12 at (189.6, 148.2)
- removed the Q12 at (129.7, 146.9)
- removed the Q13 at (180.7, 148.2)
- removed the Q13 at (129.7, 138.0)
- removed the Q14 at (171.8, 148.2)
- removed the Q14 at (129.7, 129.2)
- removed the Q15 at (198.5, 143.1)
- removed the Q15 at (134.7, 155.8)
- removed the Q16 at (189.6, 143.1)
- removed the Q16 at (134.7, 146.9)
- removed the Q17 at (180.7, 143.1)
- removed the Q17 at (134.7, 138.0)
- removed the Q18 at (171.8, 143.1)
- removed the Q18 at (134.7, 129.2)
- removed the Q2 at (238.1, 148.1)
- removed the Q2 at (129.8, 195.5)
- removed the Q3 at (229.2, 148.1)
- removed the Q3 at (129.8, 186.6)
- removed the Q4 at (220.3, 148.1)
- removed the Q4 at (129.8, 177.7)
- removed the Q5 at (211.5, 148.1)
- removed the Q5 at (129.8, 168.8)
- removed the Q6 at (238.1, 143.0)
- removed the Q6 at (134.9, 195.5)
- removed the Q7 at (229.2, 143.0)
- removed the Q7 at (134.9, 186.6)
- removed the Q8 at (220.3, 143.0)
- removed the Q8 at (134.9, 177.7)
- removed the Q9 at (211.5, 143.0)
- removed the Q9 at (134.9, 168.8)
- removed the R1 at (234.7, 148.3)
- removed the R1 at (129.6, 192.0)
- removed the R2 at (225.8, 148.3)
- removed the R2 at (129.6, 183.1)
- removed the R3 at (216.9, 148.3)
- removed the R3 at (129.6, 174.2)
- removed the R4 at (208.0, 148.3)
- removed the R4 at (129.6, 165.4)
- removed the R5 at (223.6, 171.7)
- removed the R5 at (106.2, 180.9)
- removed the R6 at (195.1, 148.4)
- removed the R6 at (129.5, 152.4)
- removed the R7 at (186.2, 148.4)
- removed the R7 at (129.5, 143.5)
- removed the R8 at (177.3, 148.4)
- removed the R8 at (129.5, 134.6)
- removed the R9 at (168.4, 148.4)
- removed the R9 at (129.5, 125.7)
- removed the U1 at (224.0, 212.9)
- removed the U1 at (80.1, 198.9)
- removed the U2 at (170.9, 168.5)
- removed the U2 at (109.3, 128.3)
- removed the U3 at (188.3, 168.5)
- removed the U3 at (109.3, 145.7)
- removed the U4 at (205.7, 168.5)
- removed the U4 at (109.3, 163.1)
- added C1: 100nF, Capacitor_SMD:C_0805_2012Metric, F.Cu at (322.7, 136.4)
- added C2: 100nF, Capacitor_SMD:C_0805_2012Metric, F.Cu at (322.7, 153.8)
- added C3: 100nF, Capacitor_SMD:C_0805_2012Metric, F.Cu at (322.7, 171.2)
- added J2: US_01_Connector, Connector_Molex:Molex_KK-254_AE-6410-04A_1x04_P2.54mm_Vertical, F.Cu at (361.2, 210.4)
- added J3: US_02_Connector, Connector_Molex:Molex_KK-254_AE-6410-04A_1x04_P2.54mm_Vertical, F.Cu at (361.2, 198.9)
- added J4: US_03, Connector_Molex:Molex_KK-254_AE-6410-04A_1x04_P2.54mm_Vertical, F.Cu at (361.2, 187.5)
- added J5: Valves, Connector_Molex:Molex_KK-254_AE-6410-05A_1x05_P2.54mm_Vertical, F.Cu at (361.2, 160.5)
- added J6: Temp_Sensor, Connector_Molex:Molex_KK-254_AE-6410-03A_1x03_P2.54mm_Vertical, F.Cu at (361.2, 171.5)
- added J7: Led Strip, Connector_Molex:Molex_KK-254_AE-6410-05A_1x05_P2.54mm_Vertical, F.Cu at (361.2, 137.2)
- added Q11: Q_NPN_BEC, Package_TO_SOT_SMD:SOT-23, F.Cu at (342.0, 146.0)
- added Q12: Q_NPN_BEC, Package_TO_SOT_SMD:SOT-23, F.Cu at (336.5, 139.6)
- added Q13: Q_NPN_BEC, Package_TO_SOT_SMD:SOT-23, F.Cu at (342.0, 135.3)
- added Q14: Q_NPN_BEC, Package_TO_SOT_SMD:SOT-23, F.Cu at (336.5, 129.0)
- added Q15: IRLML6344, Package_TO_SOT_SMD:SC-59, F.Cu at (347.1, 146.0)
- added Q16: IRLML6344, Package_TO_SOT_SMD:SC-59, F.Cu at (341.5, 139.6)
- added Q17: IRLML6344, Package_TO_SOT_SMD:SC-59, F.Cu at (347.1, 135.3)
- added Q18: IRLML6344, Package_TO_SOT_SMD:SC-59, F.Cu at (341.5, 129.0)
- added Q2: Q_NPN_BEC, Package_TO_SOT_SMD:SOT-23, F.Cu at (341.7, 169.6)
- added Q3: Q_NPN_BEC, Package_TO_SOT_SMD:SOT-23, F.Cu at (336.1, 163.2)
- added Q4: Q_NPN_BEC, Package_TO_SOT_SMD:SOT-23, F.Cu at (341.7, 158.9)
- added Q5: Q_NPN_BEC, Package_TO_SOT_SMD:SOT-23, F.Cu at (336.1, 152.6)
- added Q6: IRLML6344, Package_TO_SOT_SMD:SC-59, F.Cu at (346.8, 169.6)
- added Q7: IRLML6344, Package_TO_SOT_SMD:SC-59, F.Cu at (341.2, 163.2)
- added Q8: IRLML6344, Package_TO_SOT_SMD:SC-59, F.Cu at (346.8, 158.9)
- added Q9: IRLML6344, Package_TO_SOT_SMD:SC-59, F.Cu at (341.2, 152.6)
- added R1: 1K, Resistor_SMD:R_0805_2012Metric, F.Cu at (341.5, 166.2)
- added R2: 1K, Resistor_SMD:R_0805_2012Metric, F.Cu at (335.9, 159.8)
- added R3: 1K, Resistor_SMD:R_0805_2012Metric, F.Cu at (341.5, 155.5)
- added R4: 1K, Resistor_SMD:R_0805_2012Metric, F.Cu at (336.0, 149.1)
- added R5: 4.7k, Resistor_SMD:R_0805_2012Metric, F.Cu at (354.6, 167.7)
- added R6: 1K, Resistor_SMD:R_0805_2012Metric, F.Cu at (341.9, 142.6)
- added R7: 1K, Resistor_SMD:R_0805_2012Metric, F.Cu at (336.3, 136.2)
- added R8: 1K, Resistor_SMD:R_0805_2012Metric, F.Cu at (341.9, 131.9)
- added R9: 1K, Resistor_SMD:R_0805_2012Metric, F.Cu at (336.2, 125.5)
- added U1: NodeMCU1.0(ESP-12E), ESP8266:NodeMCU1.0(12-E), F.Cu at (328.5, 202.4)
- added U2: 74HC595, Package_SO:SOIC-16W_5.3x10.2mm_P1.27mm, F.Cu at (325.2, 129.3)
- added U3: 74HC595, Package_SO:SOIC-16W_5.3x10.2mm_P1.27mm, F.Cu at (325.2, 146.7)
- added U4: 74HC595, Package_SO:SOIC-16W_5.3x10.2mm_P1.27mm, F.Cu at (325.2, 164.1)
- moved J1 145.0 mm to (359.7, 220.5), turned to 90 degrees
- moved Q1 118.6 mm to (352.0, 220.5)
Routing:
- net +12V: track 0.00 -> 309.7 mm, vias 0 -> 9
- net +3V3: track 129.6 -> 286.4 mm, vias 0 -> 3
- net /Valve_01: track 118.9 -> 28.4 mm
- net /Valve_02: track 100.9 -> 18.7 mm
- net /Valve_04: track 89.6 -> 10.9 mm
- net /Valve_03: track 87.8 -> 20.2 mm
- net Net-(U1-Pad30): track 165.1 -> 113.7 mm
- net Net-(U1-Pad29): track 162.3 -> 112.4 mm, vias 8 -> 4
- net Net-(U1-Pad28): track 161.6 -> 112.1 mm, vias 8 -> 4
- net /Led_Red: track 68.9 -> 23.4 mm
- net /Led_Green: track 54.8 -> 13.2 mm
- net Net-(U1-Pad27): track 132.0 -> 94.5 mm, vias 8 -> 4
- net /Led_White: track 37.4 -> 6.21 mm
- net Net-(U3-Pad9): track 0.00 -> 29.7 mm, vias 0 -> 2
- net Net-(U2-Pad9): track 0.00 -> 27.7 mm
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- added copper zone on B.Cu, net GND
- added copper zone on F.Cu, net GND
Other:
- board size 190.8 x 107.7 mm -> 57.4 x 108.2 mm

Commit message: fixed names
Parts:
- J2: value US_01_Connector -> US_01
- J3: value US_02_Connector -> US_02
- J7: value Led Strip -> Led_Strip
- Q11, Q12, Q13, Q14, Q2, Q3, Q4, Q5: value Q_NPN_BEC -> NPN
