File: shema/shema.sch (KiCad schematic (older format))
At the start: 48 parts

Commit message: scheme
Parts:
- removed 100k (x3): R0805, symbol pspice:R
- removed 100k: R805, symbol pspice:R
- removed J?: Led strip connector, symbol Connector_Generic:Conn_01x05
- removed Q? (x4): IRLML6344, Package_TO_SOT_SMD:SOT-23, symbol Transistor_FET:IRLML6402
- removed Q? (x4): PNP, symbol Device:Q_PNP_Darlington_EBC
- added J?: Temp_Sensor_Connector, symbol Connector_Generic:Conn_01x03
- added J?: US_01_Connector, symbol Connector_Generic:Conn_01x04
- added J?: US_02_Connector, symbol Connector_Generic:Conn_01x04
- added J?: US_03_Connector, symbol Connector_Generic:Conn_01x04
- added R?: 4.7k, symbol Device:R
- J?: value Led_Strip_Connector -> Valves_Connector
Connections:
- net labels added: +3.3V, Temp_sensor, us_01, us_02, us_03, us_trig
- net labels removed: Temperature_Sensor
- wire segments 258 -> 234
Other:
- note added: "DQ"
- note added: "Echo"
- note added: "GND"
- note added: "LED_STRIP"
- note added: "Trig"
- note added: "Vcc"
- note added: "Vdd"
- note removed: "LED STRIP"
- note removed: "Pin 15\n"
- note removed: "Pin 1\n"
- note removed: "Pin 2\n"
- note removed: "Pin 3\n"
- moved on the sheet: C?, J?, Q?, R0805, R?, U?

Commit message: footprints
Parts:
- removed Q? (x8): IRLML6344, symbol Device:Q_NMOS_GSD
- removed Q? (x8): NPN, symbol Device:Q_NPN_CEB
- added Q10, Q15, Q16, Q17, Q18, Q6, Q7, Q8, Q9: IRLML6344, Package_TO_SOT_SMD:SC-59, symbol IRLML6344:IRLML6344TRPBFTR
- added Q11, Q12, Q13, Q14, Q2, Q3, Q4, Q5: Q_NPN_BEC, Package_TO_SOT_SMD:SOT-23, symbol Device:Q_NPN_BEC
- C1, C2: renamed from C?; footprint (none) -> Capacitor_SMD:C_0805_2012Metric
- C3: renamed from C?; footprint Capacitor_SMD:C_0805_2012Metric_Pad1.15x1.40mm_HandSolder -> Capacitor_SMD:C_0805_2012Metric
- J1: renamed from J?; footprint (none) -> TerminalBlock_4Ucon:TerminalBlock_4Ucon_1x02_P3.50mm_Vertical
- J2, J3, J4: renamed from J?; footprint (none) -> Connector_Molex:Molex_KK-254_AE-6410-04A_1x04_P2.54mm_Vertical
- J5, J7: renamed from J?; footprint (none) -> Connector_Molex:Molex_KK-254_AE-6410-05A_1x05_P2.54mm_Vertical
- J6: renamed from J?; footprint (none) -> Connector_Molex:Molex_KK-254_AE-6410-03A_1x03_P2.54mm_Vertical
- Q1: renamed from Q?; value IRLML6344 -> IRLML6402; footprint Package_TO_SOT_SMD:SOT-23 -> Package_TO_SOT_SMD:SC-59
- R1, R2, R3, R4, R5: renamed from R?; footprint (none) -> Resistor_SMD:R_0805_2012Metric
- R6, R7, R8, R9: renamed from R0805; footprint (none) -> Resistor_SMD:R_0805_2012Metric
- U1: renamed from U?; footprint (none) -> ESP8266:NodeMCU1.0(12-E)
- U2, U3, U4: renamed from U?; footprint (none) -> Package_SO:SOIC-16W_5.3x10.2mm_P1.27mm
Connections:
- net GND: now also Q11.2 (E), Q12.2 (E), Q13.2 (E), Q14.2 (E), Q15.2 (S), Q16.2 (S), Q17.2 (S), Q18.2 (S), Q2.2 (E), Q3.2 (E), Q4.2 (E), Q5.2 (E), Q6.2 (S), Q7.2 (S), Q8.2 (S), Q9.2 (S)
- net Led_Blue: now also Q13.1 (B)
- net Led_Green: now also Q12.1 (B)
- net Led_Red: now also Q11.1 (B)
- net Led_White: now also Q14.1 (B)
- net Valve_01: now also Q2.1 (B)
- net Valve_02: now also Q3.1 (B)
- net Valve_03: now also Q4.1 (B)
- net Valve_04: now also Q5.1 (B)
- net at J7.2 (Pin_2): now also Q15.3 (D)
- net at J7.3 (Pin_3): now also Q16.3 (D)
- net at J7.4 (Pin_4): now also Q17.3 (D)
- net at J7.5 (Pin_5): now also Q18.3 (D)
- net at R6.2: now also Q11.3 (C), Q15.1 (G)
- net at R7.2: now also Q12.3 (C), Q16.1 (G)
- net at R8.2: now also Q13.3 (C), Q17.1 (G)
- net at R9.2: now also Q14.3 (C), Q18.1 (G)
- net at J5.2 (Pin_2): now also Q6.3 (D)
- net at J5.3 (Pin_3): now also Q7.3 (D)
- net at J5.4 (Pin_4): now also Q8.3 (D)
- net at J5.5 (Pin_5): now also Q9.3 (D)
- net at R1.2: now also Q2.3 (C), Q6.1 (G)
- net at R2.2: now also Q3.3 (C), Q7.1 (G)
- net at R3.2: now also Q4.3 (C), Q8.1 (G)
- net at R4.2: now also Q5.3 (C), Q9.1 (G)
Other:
- note removed: "Pin 1"
- note removed: "Pin 15"
- note removed: "Pin 2"
- note removed: "Pin 3"
- moved on the sheet: J6, R5

Commit message: first steps
Connections:
- net Cooling: now also U3.5 (QF); no longer U2.7 (QH)
- net Heater_01: now also U2.2 (QC); no longer U2.5 (QF)
- net Heater_02: now also U2.1 (QB); no longer U2.6 (QG)
- net Led_Blue: now also U2.5 (QF); no longer U2.2 (QC)
- net Led_Green: now also U2.6 (QG); no longer U2.1 (QB)
- net Led_Red: now also U2.7 (QH); no longer U2.15 (QA)
- net Led_White: now also U2.4 (QE); no longer U2.3 (QD)
- net Valve_01: now also U3.4 (QE); no longer U3.15 (QA)
- net Valve_02: now also U3.3 (QD); no longer U3.1 (QB)
- net Valve_04: now also U3.1 (QB); no longer U3.3 (QD)
- net Water_Pump: now also U2.3 (QD); no longer U2.4 (QE)
- net Wave_Maker: now also U3.15 (QA); no longer U3.4 (QE)
- net at U2.12 (RCLK), U3.12 (RCLK), U4.12 (RCLK): now also U1.28 (D2(GPIO4)); no longer U1.27 (D3(GPIO0))
- net at U2.10 (~SRCLR), U3.10 (~SRCLR), U4.10 (~SRCLR): now also U1.30 (D0(GPIO16)); no longer U1.28 (D2(GPIO4))
- net at U2.14 (SER): now also U1.27 (D3(GPIO0)); no longer U1.30 (D0(GPIO16))
Changed lines of the file:
@@
 Wire Wire Line
 	3750 5250 3000 5250
-Wire Wire Line
-	2950 3000 2950 7850
-Wire Wire Line
-	2950 7850 2850 7850
-Wire Wire Line
-	3000 7950 2850 7950
-Wire Wire Line
-	3050 8050 2850 8050
-Wire Wire Line
-	3100 8150 2850 8150
 NoConn ~ 4550 8000
-Text Label 5200 3000 2    50   ~ 0
+Text Label 5200 3700 2    50   ~ 0
 Led_Red
-Text Label 5200 3100 2    50   ~ 0
+Text Label 5200 3600 2    50   ~ 0
 Led_Green
-Text Label 5200 3200 2    50   ~ 0
+Text Label 5200 3500 2    50   ~ 0
 Led_Blue
+Text Label 5200 3400 2    50   ~ 0
+Led_White
 Text Label 5200 3300 2    50   ~ 0
-Led_White
-Text Label 5200 3400 2    50   ~ 0
 Water_Pump
-Text Label 5200 5050 2    50   ~ 0
+Text Label 5200 5450 2    50   ~ 0
 Valve_01
-Text Label 5200 5150 2    50   ~ 0
+Text Label 5200 5350 2    50   ~ 0
 Valve_02
 Text Label 5200 5250 2    50   ~ 0
 Valve_03
-Text Label 5200 5350 2    50   ~ 0
+Text Label 5200 5150 2    50   ~ 0
 Valve_04
-Text Label 5200 3500 2    50   ~ 0
+Text Label 5200 3200 2    50   ~ 0
 Heater_01
-Text Label 5200 3600 2    50   ~ 0
+Text Label 5200 3100 2    50   ~ 0
 Heater_02
-Text Label 5200 3700 2    50   ~ 0
+Text Label 5200 5550 2    50   ~ 0
 Cooling
-Text Label 5200 5450 2    50   ~ 0
+Text Label 5200 5050 2    50   ~ 0
 Wave_Maker
 Text Label 800  7850 0    50   ~ 0
@@
 	13400 5950 13400 5850
 Connection ~ 13400 5950
-Wire Wire Line
-	5200 3000 4550 3000
 Text Label 3400 8250 2    50   ~ 0
 Temp_sensor
@@
 Wire Wire Line
 	3000 7300 3000 7950
-Wire Wire Line
-	3050 7400 3050 8050
-Wire Wire Line
-	3100 7600 3100 8150
 $Comp
 L Connector_Generic:Conn_01x03 J6
@@
 	1    0    0    -1
 $EndComp
+Wire Wire Line
+	4550 5550 5200 5550
+Wire Wire Line
+	3000 7950 2850 7950
+Wire Wire Line
+	3050 7850 2850 7850
+Wire Wire Line
+	3050 7400 3050 7850
+Wire Wire Line
+	3100 8050 2850 8050
+Wire Wire Line
+	3100 7600 3100 8050
+Wire Wire Line
+	2950 3000 2950 8150
+Wire Wire Line
+	2950 8150 2850 8150
 $EndSCHEMATC

Commit message: temp sensor pcb
Parts:
- removed Q10: IRLML6344, Package_TO_SOT_SMD:SC-59, symbol IRLML6344:IRLML6344TRPBFTR
Connections:
- net Heater_01: now also U2.6 (QG); no longer U2.2 (QC)
- net Heater_02: now also U2.7 (QH); no longer U2.1 (QB)
- net Led_Blue: now also U2.3 (QD); no longer U2.5 (QF)
- net Led_Green: now also U2.2 (QC); no longer U2.6 (QG)
- net Led_Red: now also U2.1 (QB); no longer U2.7 (QH)
- net Valve_01: now also U3.1 (QB); no longer U3.4 (QE)
- net Valve_02: now also U3.2 (QC); no longer U3.3 (QD)
- net Valve_03: now also U3.3 (QD); no longer U3.2 (QC)
- net Valve_04: now also U3.4 (QE); no longer U3.1 (QB)
- net Water_Pump: now also U2.5 (QF); no longer U2.3 (QD)
- net Wave_Maker: now also U3.6 (QG); no longer U3.15 (QA)
Other:
- moved on the sheet: J5, Q2, Q3, Q4, Q5, Q6, Q7, Q8, Q9, R1, R2, R3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

Commit message: second version
Connections:
- net Flowmeter: now also U1.4 (SD3(GPIO10)); no longer U1.23 (D5(GPIO14))
- net us_01: now also U1.20 (D8(GPIO15)); no longer U1.22 (D6(GPIO12))
- net us_03: now also U1.22 (D6(GPIO12)); no longer U1.20 (D8(GPIO15))
- net us_trig: now also U1.23 (D5(GPIO14)); no longer U1.4 (SD3(GPIO10))
Changed lines of the file:
@@
 Text Label 800  7850 0    50   ~ 0
 PH_Sensor
-Text Label 3400 8550 2    50   ~ 0
+Text Label 800  8150 0    50   ~ 0
 Flowmeter
 Text Label 17900 9050 0    50   ~ 0
@@
 Wire Wire Line
 	800  8150 1250 8150
-Text Label 800  8150 0    50   ~ 0
+Text Label 3400 8550 2    50   ~ 0
 us_trig
-Text Label 3400 8650 2    50   ~ 0
+Text Label 3400 8850 2    50   ~ 0
 us_01
 Wire Wire Line
@@
 Text Label 3400 8750 2    50   ~ 0
 us_02
-Text Label 3400 8850 2    50   ~ 0
+Text Label 3400 8650 2    50   ~ 0
 us_03
 Wire Wire Line

Commit message: arduino web server
Parts:
- Q15, Q16, Q17, Q18, Q6, Q7, Q8, Q9: symbol IRLML6344:IRLML6344TRPBFTR -> shema-rescue:IRLML6344TRPBFTR-IRLML6344
Changed lines of the file:
@@
 $EndComp
 $Comp
-L IRLML6344:IRLML6344TRPBFTR Q15
+L shema-rescue:IRLML6344TRPBFTR-IRLML6344 Q15
 U 1 1 5C8B9D41
 P 14050 1750
@@
 	14800 1300 14800 5200
 $Comp
-L IRLML6344:IRLML6344TRPBFTR Q16
+L shema-rescue:IRLML6344TRPBFTR-IRLML6344 Q16
 U 1 1 5C8D16A1
 P 14050 3150
@@
 $EndComp
 $Comp
-L IRLML6344:IRLML6344TRPBFTR Q18
+L shema-rescue:IRLML6344TRPBFTR-IRLML6344 Q18
 U 1 1 5C8D1FD5
 P 14050 5950
@@
 $EndComp
 $Comp
-L IRLML6344:IRLML6344TRPBFTR Q17
+L shema-rescue:IRLML6344TRPBFTR-IRLML6344 Q17
 U 1 1 5C8D2062
 P 14050 4550
@@
 $EndComp
 $Comp
-L IRLML6344:IRLML6344TRPBFTR Q6
+L shema-rescue:IRLML6344TRPBFTR-IRLML6344 Q6
 U 1 1 5C8D56D0
 P 10250 2000
@@
 $EndComp
 $Comp
-L IRLML6344:IRLML6344TRPBFTR Q7
+L shema-rescue:IRLML6344TRPBFTR-IRLML6344 Q7
 U 1 1 5C8D8F1A
 P 10250 3400
@@
 $EndComp
 $Comp
-L IRLML6344:IRLML6344TRPBFTR Q8
+L shema-rescue:IRLML6344TRPBFTR-IRLML6344 Q8
 U 1 1 5C8D9954
 P 10250 4800
@@
 $EndComp
 $Comp
-L IRLML6344:IRLML6344TRPBFTR Q9
+L shema-rescue:IRLML6344TRPBFTR-IRLML6344 Q9
 U 1 1 5C91FFC3
 P 10250 6200
